File: Hardware/Qwiic Proximity Sensor - VCNL4040.brd (EAGLE design)
At the start: 25.4 x 25.4 mm, 42 parts, among them J2 SMD, J3 PTH, J4 SMD, U2 VCNL4040

Commit message: post checklist changes
Parts:
- added U$8: (no value), buzzard_labels (27):ADDR_0X600
- J2, J4: value SMD -> (none); device SparkX:1X04_1MM_RA -> SparkFun-Connectors:1X04_1MM_RA
- moved LOGO2 31.8 mm to (-8.89, -20.3)
- moved R1 0.63 mm to (7.62, 12.1)
- moved U$19 0.13 mm to (6.73, 19.7)
Routing:
- net !INT: track 25.9 -> 24.8 mm
- net GND: track 4.29 -> 4.22 mm, vias 7 -> 11
Other:
- board text added: "Andy England"
- board text added: "Nathan Seidle"
- board text added: "v10"
- board text removed: "v01"
