File: Hardware/Qwiic Proximity Sensor - VCNL4040.sch (EAGLE design)
At the start: 25 parts, among them J2 SMD, J3 PTH, J4 SMD, U2 VCNL4040

Commit message: post checklist changes
Parts:
- J2, J4: value SMD -> (none); device SparkX:I2C_STANDARDJS-1MM -> SparkFun-Connectors:QWIIC_CONNECTORJS-1MM
Connections:
- net 3.3V: now also J2.2, J4.2; no longer J2.VCC, J4.VCC
- net GND: now also J2.1, J4.1; no longer J2.GND, J4.GND
- net SCL: now also J2.4, J4.4; no longer J2.SCL, J4.SCL
- net SDA: now also J2.3, J4.3; no longer J2.SDA, J4.SDA
Other:
- note added: "VIN: 2.5V-3.6V"
- note added: "v10"
- note removed: "v01"
Changed lines of the file:
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@@
 <part name="SUPPLY1" library="SparkFun-PowerSymbols" deviceset="3.3V" device=""/>
 <part name="SUPPLY4" library="SparkFun-PowerSymbols" deviceset="3.3V" device=""/>
-<part name="J2" library="SparkX" deviceset="I2C_STANDARD" device="JS-1MM" value="SMD"/>
+<part name="J2" library="SparkFun-Connectors" deviceset="QWIIC_CONNECTOR" device="JS-1MM"/>
 <part name="GND6" library="SparkFun" deviceset="GND" device=""/>
 <part name="SUPPLY7" library="SparkFun-PowerSymbols" deviceset="3.3V" device=""/>
@@
 <part name="U$2" library="SparkFun-Aesthetics" deviceset="SFE_LOGO_NAME_FLAME" device=".1_INCH"/>
 <part name="SUPPLY8" library="SparkFun-PowerSymbols" deviceset="3.3V" device=""/>
-<part name="J4" library="SparkX" deviceset="I2C_STANDARD" device="JS-1MM" value="SMD"/>
+<part name="J4" library="SparkFun-Connectors" deviceset="QWIIC_CONNECTOR" device="JS-1MM"/>
 <part name="GND8" library="SparkFun" deviceset="GND" device=""/>
 <part name="LOGO1" library="SparkFun-Aesthetics" deviceset="OSHW-LOGO" device="MINI"/>
@@
 <plain>
 <text x="167.894" y="11.43" size="2.54" layer="94" font="vector">N. Seidle</text>
-<text x="237.744" y="7.366" size="2.54" layer="94" font="vector">v01</text>
+<text x="237.744" y="7.366" size="2.54" layer="94" font="vector">v10</text>
 <text x="91.44" y="86.36" size="1.778" layer="97" font="vector">7-bit unshifted I2C address: 0x60</text>
 <text x="165.1" y="134.62" size="1.778" layer="97" font="vector">Clear I2C Jumper to remove
@@
 <text x="64.262" y="60.452" size="3.048" layer="97" font="vector">Connections</text>
 <text x="169.418" y="7.112" size="2.54" layer="94" font="vector">A. England</text>
+<text x="84.582" y="156.464" size="1.778" layer="97" font="vector">VIN: 2.5V-3.6V</text>
 </plain>
 <instances>
@@
 </segment>
 <segment>
-<pinref part="J2" gate="G$1" pin="VCC"/>
+<pinref part="J2" gate="G$1" pin="2"/>
 <wire x1="63.5" y1="35.56" x2="60.96" y2="35.56" width="0.1524" layer="91"/>
 <wire x1="60.96" y1="35.56" x2="60.96" y2="43.18" width="0.1524" layer="91"/>
@@
 </segment>
 <segment>
-<pinref part="J4" gate="G$1" pin="VCC"/>
+<pinref part="J4" gate="G$1" pin="2"/>
 <wire x1="38.1" y1="35.56" x2="35.56" y2="35.56" width="0.1524" layer="91"/>
 <wire x1="35.56" y1="35.56" x2="35.56" y2="43.18" width="0.1524" layer="91"/>
@@
 <net name="GND" class="0">
 <segment>
-<pinref part="J2" gate="G$1" pin="GND"/>
+<pinref part="J2" gate="G$1" pin="1"/>
 <wire x1="63.5" y1="33.02" x2="60.96" y2="33.02" width="0.1524" layer="91"/>
 <wire x1="60.96" y1="33.02" x2="60.96" y2="30.48" width="0.1524" layer="91"/>
@@
 </segment>
 <segment>
-<pinref part="J4" gate="G$1" pin="GND"/>
+<pinref part="J4" gate="G$1" pin="1"/>
 <wire x1="38.1" y1="33.02" x2="35.56" y2="33.02" width="0.1524" layer="91"/>
 <wire x1="35.56" y1="33.02" x2="35.56" y2="30.48" width="0.1524" layer="91"/>
@@
 <net name="SCL" class="0">
 <segment>
-<pinref part="J2" gate="G$1" pin="SCL"/>
+<pinref part="J2" gate="G$1" pin="4"/>
 <wire x1="63.5" y1="40.64" x2="58.42" y2="40.64" width="0.1524" layer="91"/>
 <label x="58.42" y="40.64" size="1.27" layer="95" font="vector" rot="R180" xref="yes"/>
@@
 </segment>
 <segment>
-<pinref part="J4" gate="G$1" pin="SCL"/>
+<pinref part="J4" gate="G$1" pin="4"/>
 <wire x1="38.1" y1="40.64" x2="33.02" y2="40.64" width="0.1524" layer="91"/>
 <label x="33.02" y="40.64" size="1.27" layer="95" font="vector" rot="R180" xref="yes"/>
@@
 <net name="SDA" class="0">
 <segment>
-<pinref part="J2" gate="G$1" pin="SDA"/>
+<pinref part="J2" gate="G$1" pin="3"/>
 <wire x1="63.5" y1="38.1" x2="58.42" y2="38.1" width="0.1524" layer="91"/>
 <label x="58.42" y="38.1" size="1.27" layer="95" font="vector" rot="R180" xref="yes"/>
@@
 </segment>
 <segment>
-<pinref part="J4" gate="G$1" pin="SDA"/>
+<pinref part="J4" gate="G$1" pin="3"/>
 <wire x1="38.1" y1="38.1" x2="33.02" y2="38.1" width="0.1524" layer="91"/>
 <label x="33.02" y="38.1" size="1.27" layer="95" font="vector" rot="R180" xref="yes"/>
